Commit message: feat: new basketbot model

File: basketbot/urdf/basketbot.1.xacro (robot description, xacro)
@@ -1,15 +1,15 @@
 <?xml version="1.0"?>
 <robot name="basketbot" xmlns:xacro="http://www.ros.org/wiki/xacro">
-  <!--<xacro:include filename="$(find basketbot)/urdf/basketbot.gazebo" />-->
+  <xacro:include filename="$(find basketbot)/urdf/basketbot.gazebo" />
   <!--  VARIABLES -->
   <xacro:property name="chassis_length" value="1.1" />
   <xacro:property name="chassis_width" value="0.84" />
-  <xacro:property name="chassis_height" value="0.85" />
-  <xacro:property name="wheel_length" value="0.05" />
-  <xacro:property name="wheel_radius" value="0.15" />
-  <xacro:property name="wheel_mass" value="0.25" />
-  <xacro:property name="wheel_x_offset" value="0.35" />
+  <xacro:property name="chassis_height" value="0.2" />
+  <xacro:property name="wheel_length" value="0.152" />
+  <xacro:property name="wheel_radius" value="0.463" />
+  <xacro:property name="wheel_mass" value=".25" />
+  <xacro:property name="wheel_x_offset" value="0.09" />
   <xacro:property name="wheel_y_offset" value="${(chassis_width/2) + (wheel_length/2)}" />
-  <xacro:property name="wheel_z_offset" value="-0.3175" />
+  <xacro:property name="wheel_z_offset" value="-${chassis_height * 0.25}" />
   <xacro:property name="wheel_rpy" value="0 ${pi/2} ${pi/2}" />
   <xacro:property name="wheel_front_joint_xyz" value="0 0 0" />
@@ -29,5 +29,5 @@
   </joint>
   <link name="chassis">
-    <pose>0 0 0 0 0 0</pose>
+    <pose>0 0 0.1 0 0 0</pose>
     <inertial>
       <mass value="15.0" />
@@ -48,9 +48,69 @@
       <origin xyz="0 0 0" rpy="0 0 0" />
       <geometry>
-        <mesh filename="package://basketbot/meshes/BasketBotModel.dae" />
-      </geometry>
-    </visual>
-  </link>
+        <box size="${chassis_length} ${chassis_width} ${chassis_height}" />
+<!--        <mesh filename="package://basketbot/meshes/BasketBotModel.dae" /> -->
+      </geometry>
+    </visual>
+  </link>
+<!--
+  <joint name="body_joint" type="fixed">
+    <origin xyz="-0.05 0 ${chassis_height - wheel_z_offset}" rpy=" 0 0 0" />
+    <parent link="chassis" />
+    <child link="body" />
+  </joint>
+  <link name="body">
+    <collision name='body_collision'>
+      <origin xyz="0 0 0" rpy=" 0 0 0" />
+      <geometry>
+        <box size="${chassis_length *0.75} ${chassis_width*0.75} ${chassis_height*1.5}" />
+      </geometry>
+    </collision>
+    <visual name='body_visual'>
+      <origin xyz="0 0 0" rpy=" 0 0 0" />
+      <geometry>
+        <box size="${chassis_length *0.75} ${chassis_width*0.75} ${chassis_height*1.5}" />
+      </geometry>
+    </visual>
+    <inertial>
+      <mass value="1.0" />
+      <origin xyz="0.0 0 0" rpy="0 0 0" />
+      <inertia
+        ixx="0.1" ixy="0" ixz="0"
+        iyy="0.1" iyz="0"
+        izz="0.1"
+      />
+    </inertial>
+  </link>
+  <joint name="body_fairing_joint" type="fixed">
+    <origin xyz="0.075 0  ${chassis_height - wheel_z_offset}" rpy=" 0 0 0" />
+    <parent link="chassis" />
+    <child link="body_fairing" />
+  </joint>
+  <link name="body_fairing">
+    <collision name='body_fairing_collision'>
+      <origin xyz="0 0 0" rpy="0 0 0" />
+      <geometry>
+        <sphere radius="${chassis_width*0.5*0.75}" />
+      </geometry>
+    </collision>
+    <visual name='body_fairing_visual'>
+      <origin xyz="0 0 0" rpy="0 0 0" />
+      <geometry>
+        <sphere radius="${chassis_width*0.5*0.75}" />
+      </geometry>
+    </visual>
+    <inertial>
+      <mass value="0.25" />
+      <origin xyz="0.0 0 0" rpy="0 0 0" />
+      <inertia
+        ixx="0.1" ixy="0" ixz="0"
+        iyy="0.1" iyz="0"
+        izz="0.1"
+      />
+    </inertial>
+  </link>
+-->
   <!--  WHEELS  -->
+  <!--
   <joint type="continuous" name="wheel_left_front_joint">
     <origin xyz="${wheel_x_offset} ${wheel_y_offset} ${wheel_z_offset}" rpy="0 0 0"/>
@@ -93,39 +153,5 @@
     </visual>
     <collision name="wheel_left_front_collision">
-      <origin xyz="0.0 0 0" rpy="0 0 ${pi}" />
-      <geometry>
-        <cylinder radius="${wheel_radius}" length="${wheel_length}" />
-      </geometry>
-      <surface>
-        <friction>
-          <fdir1>1 0 0</fdir1>
-          <kp>${wheel_kp}</kp>
-          <kd>${wheel_kd}</kd>
-          <mu>${wheel_mu1}</mu>
-          <mu2>${wheel_mu2}</mu2>
-          <slip1>${wheel_slip1}</slip1>
-          <slip2>${wheel_slip2}</slip2>
-        </friction>
-      </surface>
-    </collision>
-    <inertial>
-      <mass value="${wheel_mass}" />
-      <origin xyz="0.0 0 0" rpy="0 0 ${pi}" />
-      <inertia
-        ixx="${wheel_inertia}" ixy="0" ixz="0"
-        iyy="${wheel_inertia}" iyz="0"
-        izz="${wheel_inertia}"
-      />
-    </inertial>
-  </link>
-  <link name="wheel_left_rear">
-    <visual name="wheel_left_rear_visual">
-      <origin xyz="0.0 0 0" rpy="0 0 ${pi}" />
-      <geometry>
-        <mesh filename="package://basketbot/meshes/wheel.dae" />
-      </geometry>
-    </visual>
-    <collision name="wheel_left_rear_collision">
-      <origin xyz="0.0 0 0" rpy="0 0 ${pi}" />
+      <origin xyz="0.0 0 0" rpy="${wheel_rpy}" />
       <geometry>
         <cylinder radius="${wheel_radius}" length="${wheel_length}" />
@@ -153,13 +179,13 @@
     </inertial>
   </link>
-  <link name="wheel_right_front">
-    <visual name="wheel_right_front_visual">
-      <origin xyz="0.0 0 0" rpy="0 0 -${pi}" />
-      <geometry>
-      <mesh filename="package://basketbot/meshes/wheel.dae" />
-      </geometry>
-    </visual>
-    <collision name="wheel_right_front_collision">
-      <origin xyz="0.0 0 0" rpy="0 0 -${pi}" />
+  <link name="wheel_left_rear">
+    <visual name="wheel_left_rear_visual">
+      <origin xyz="0.0 0 0" rpy="${wheel_rpy}" />
+      <geometry>
+        <mesh filename="package://basketbot/meshes/wheel.dae" />
+      </geometry>
+    </visual>
+    <collision name="wheel_left_rear_collision">
+      <origin xyz="0.0 0 0" rpy="${wheel_rpy}" />
       <geometry>
         <cylinder radius="${wheel_radius}" length="${wheel_length}" />
@@ -179,5 +205,5 @@
     <inertial>
       <mass value="${wheel_mass}" />
-      <origin xyz="0.0 0 0" rpy="0 0 -${pi}" />
+      <origin xyz="0.0 0 0" rpy="${wheel_rpy}" />
       <inertia
         ixx="${wheel_inertia}" ixy="0" ixz="0"
@@ -187,13 +213,13 @@
     </inertial>
   </link>
-  <link name="wheel_right_rear">
-    <visual name="wheel_right_rear_visual">
-      <origin xyz="0.0 0 0" rpy="0 0 -${pi}" />
-      <geometry>
-        <mesh filename="package://basketbot/meshes/wheel.dae" />
-      </geometry>
-    </visual>
-    <collision name="wheel_right_rear_collision">
-      <origin xyz="0.0 0 0" rpy="0 0 -${pi}" />
+  <link name="wheel_right_front">
+    <visual name="wheel_right_front_visual">
+      <origin xyz="0.0 0 0" rpy="${wheel_rpy}" />
+      <geometry>
+        <cylinder radius="${wheel_radius}" length="${wheel_length}" />
+      </geometry>
+    </visual>
+    <collision name="wheel_right_front_collision">
+      <origin xyz="0.0 0 0" rpy="${wheel_rpy}" />
       <geometry>
         <cylinder radius="${wheel_radius}" length="${wheel_length}" />
@@ -213,5 +239,5 @@
     <inertial>
       <mass value="${wheel_mass}" />
-      <origin xyz="0.0 0 0" rpy="0 0 -${pi}" />
+      <origin xyz="0.0 0 0" rpy="${wheel_rpy}" />
       <inertia
         ixx="${wheel_inertia}" ixy="0" ixz="0"
@@ -221,3 +247,127 @@
     </inertial>
   </link>
+  <link name="wheel_right_rear">
+    <visual name="wheel_right_rear_visual">
+      <origin xyz="0.0 0 0" rpy="${wheel_rpy}" />
+      <geometry>
+        <cylinder radius="${wheel_radius}" length="${wheel_length}" />
+      </geometry>
+    </visual>
+    <collision name="wheel_right_rear_collision">
+      <origin xyz="0.0 0 0" rpy="${wheel_rpy}" />
+      <geometry>
+        <cylinder radius="${wheel_radius}" length="${wheel_length}" />
+      </geometry>
+      <surface>
+        <friction>
+          <fdir1>1 0 0</fdir1>
+          <kp>${wheel_kp}</kp> <!-- kp and kd for rubber -->
+          <kd>${wheel_kd}</kd>
+          <mu>${wheel_mu1}</mu>
+          <mu2>${wheel_mu2}</mu2>
+          <slip1>${wheel_slip1}</slip1>
+          <slip2>${wheel_slip2}</slip2>
+        </friction>
+      </surface>
+    </collision>
+    <inertial>
+      <mass value="${wheel_mass}" />
+      <origin xyz="0.0 0 0" rpy="${wheel_rpy}" />
+      <inertia
+        ixx="${wheel_inertia}" ixy="0" ixz="0"
+        iyy="${wheel_inertia}" iyz="0"
+        izz="${wheel_inertia}"
+      />
+    </inertial>
+  </link>
+-->
+  <!-- SENSORS  -->
+<!--
+  <joint type="fixed" name="camera_joint">
+    <origin xyz=".2 0 0" rpy="0 0 0" />
+    <child link="camera" />
+    <parent link="chassis" />
+    <axis xyz="0 1 0" />
+  </joint>
+  <link name="camera">
+    <visual name="camera_visual">
+      <origin xyz="0 0 0" rpy="0 0 0"/>
+      <geometry>
+        <box size="0.05 0.05 0.05" />
+      </geometry>
+    </visual>
+    <collision name="camera_collision">
+      <origin xyz="0 0 0" rpy="0 0 0" />
+      <geometry>
+        <box size="0.05 0.05 0.05" />
+      </geometry>
+    </collision>
+    <inertial>
+      <mass value="0.1" />
+      <origin xyz="0 0 0" rpy="0 0 0" />
+      <box_inertia m="0.1" x="0.05" y="0.05" z="0.05" />
+      <inertia
+        ixx="1e-6" ixy="0" ixz="0"
+        iyy="1e-6" iyz="0"
+        izz="1e-6"
+      />
+    </inertial>
+  </link>
+  <joint type="fixed" name="hokuyo_joint">
+    <origin xyz="0.175 0 0.08" rpy="0 0 0" />
+    <child link="hokuyo" />
+    <parent link="chassis" />
+    <axis xyz="0 1 0" />
+  </joint>
+  <link name="hokuyo">
+    <visual name="hokuyo_visual">
+      <origin xyz="0 0 0" rpy="0 0 0" />
+      <geometry>
+        <mesh filename="package://basketbot/meshes/hokuyo.dae" />
+      </geometry>
+    </visual>
+    <collision name="hokuyo_collision">
+      <origin xyz="0 0 0" rpy="0 0 0" />
+      <geometry>
+        <box size="0.1 0.1 0.1" />
+      </geometry>
+    </collision>
+    <inertial>
+      <mass value="1e-5" />
+      <origin xyz="0 0 0" rpy="0 0 0" />
+      <inertia
+        ixx="1e-6" ixy="0" ixz="0"
+        iyy="1e-6" iyz="0"
+        izz="1e-6"
+      />
+    </inertial>
+  </link>
+-->
+  <!--  COLOURS  -->
+<!--
+  <gazebo reference="chassis">
+    <material>Gazebo/Yellow</material>
+  </gazebo>
+  <gazebo reference="body">
+    <material>Gazebo/BlueGlow</material>
+  </gazebo>
+  <gazebo reference="body_fairing">
+    <material>Gazebo/BlueGlow</material>
+  </gazebo>
+  <gazebo reference="wheel_left_front">
+    <material>Gazebo/Black</material>
+  </gazebo>
+  <gazebo reference="wheel_left_rear">
+    <material>Gazebo/Black</material>
+  </gazebo>
+  <gazebo reference="wheel_right_front">
+    <material>Gazebo/Black</material>
+  </gazebo>
+  <gazebo reference="wheel_right_rear">
+    <material>Gazebo/Black</material>
+  </gazebo>
+  <gazebo reference="camera">
+    <material>Gazebo/Red</material>
+  </gazebo>
+-->
 </robot>
