Commit message: fix: rename my_robot to basketbot in all relevant files

File: basketbot/urdf/basketbot.xacro (robot description, xacro)
@@ -1,5 +1,5 @@
 <?xml version="1.0"?>
-<robot name="my_robot" xmlns:xacro="http://www.ros.org/wiki/xacro">
-  <xacro:include filename="$(find my_robot)/urdf/my_robot.gazebo" />
+<robot name="basketbot" xmlns:xacro="http://www.ros.org/wiki/xacro">
+  <xacro:include filename="$(find basketbot)/urdf/basketbot.gazebo" />
   <!--  VARIABLES -->
   <xacro:property name="chassis_length" value="0.4" />
@@ -318,5 +318,5 @@
       <origin xyz="0 0 0" rpy="0 0 0" />
       <geometry>
-        <mesh filename="package://my_robot/meshes/hokuyo.dae" />
+        <mesh filename="package://basketbot/meshes/hokuyo.dae" />
       </geometry>
     </visual>

Commit message: feat: new simplified basketbot model

File: basketbot/urdf/basketbot.xacro (robot description, xacro)
@@ -1,5 +1,5 @@
 <?xml version="1.0"?>
 <robot name="basketbot" xmlns:xacro="http://www.ros.org/wiki/xacro">
-  <!--<xacro:include filename="$(find basketbot)/urdf/basketbot.gazebo" />-->
+  <xacro:include filename="$(find basketbot)/urdf/basketbot.gazebo" />
   <!--  VARIABLES -->
   <xacro:property name="chassis_length" value="1.1" />
@@ -7,11 +7,9 @@
   <xacro:property name="chassis_height" value="0.85" />
   <xacro:property name="wheel_length" value="0.05" />
-  <xacro:property name="wheel_radius" value="0.15" />
+  <xacro:property name="wheel_radius" value="0.075" />
   <xacro:property name="wheel_mass" value="0.25" />
   <xacro:property name="wheel_x_offset" value="0.35" />
   <xacro:property name="wheel_y_offset" value="${(chassis_width/2) + (wheel_length/2)}" />
-  <xacro:property name="wheel_z_offset" value="-0.3175" />
-  <xacro:property name="wheel_rpy" value="0 ${pi/2} ${pi/2}" />
-  <xacro:property name="wheel_front_joint_xyz" value="0 0 0" />
+  <xacro:property name="wheel_z_offset" value="-0.34" />
   <xacro:property name="wheel_inertia" value="0.1" />
   <xacro:property name="wheel_kp" value="1000000.0" />
@@ -48,4 +46,5 @@
       <origin xyz="0 0 0" rpy="0 0 0" />
       <geometry>
+      <!--<box size="${chassis_length} ${chassis_width} ${chassis_height}" />-->
         <mesh filename="package://basketbot/meshes/BasketBotModel.dae" />
       </geometry>
@@ -90,4 +89,5 @@
       <geometry>
         <mesh filename="package://basketbot/meshes/wheel.dae" />
+        <cylinder radius="${wheel_radius}" length="${wheel_length}" />
       </geometry>
     </visual>
@@ -134,16 +134,16 @@
         <friction>
           <fdir1>1 0 0</fdir1>
-          <kp>${wheel_kp}</kp> <!-- kp and kd for rubber -->
-          <kd>${wheel_kd}</kd>
-          <mu>${wheel_mu1}</mu>
-          <mu2>${wheel_mu2}</mu2>
-          <slip1>${wheel_slip1}</slip1>
-          <slip2>${wheel_slip2}</slip2>
-        </friction>
-      </surface>
-    </collision>
-    <inertial>
-      <mass value="${wheel_mass}" />
-      <origin xyz="0.0 0 0" rpy="${wheel_rpy}" />
+          <kp>${wheel_kp}</kp>
+          <kd>${wheel_kd}</kd>
+          <mu>${wheel_mu1}</mu>
+          <mu2>${wheel_mu2}</mu2>
+          <slip1>${wheel_slip1}</slip1>
+          <slip2>${wheel_slip2}</slip2>
+        </friction>
+      </surface>
+    </collision>
+    <inertial>
+      <mass value="${wheel_mass}" />
+      <origin xyz="0.0 0 0" rpy="0 0 -${pi}" />
       <inertia
         ixx="${wheel_inertia}" ixy="0" ixz="0"
@@ -155,5 +155,5 @@
   <link name="wheel_right_front">
     <visual name="wheel_right_front_visual">
-      <origin xyz="0.0 0 0" rpy="0 0 -${pi}" />
+      <origin xyz="0.0 0 0" rpy="0 0 ${pi}" />
       <geometry>
       <mesh filename="package://basketbot/meshes/wheel.dae" />
@@ -161,23 +161,23 @@
     </visual>
     <collision name="wheel_right_front_collision">
-      <origin xyz="0.0 0 0" rpy="0 0 -${pi}" />
-      <geometry>
-        <cylinder radius="${wheel_radius}" length="${wheel_length}" />
-      </geometry>
-      <surface>
-        <friction>
-          <fdir1>1 0 0</fdir1>
-          <kp>${wheel_kp}</kp> <!-- kp and kd for rubber -->
-          <kd>${wheel_kd}</kd>
-          <mu>${wheel_mu1}</mu>
-          <mu2>${wheel_mu2}</mu2>
-          <slip1>${wheel_slip1}</slip1>
-          <slip2>${wheel_slip2}</slip2>
-        </friction>
-      </surface>
-    </collision>
-    <inertial>
-      <mass value="${wheel_mass}" />
-      <origin xyz="0.0 0 0" rpy="0 0 -${pi}" />
+      <origin xyz="0.0 0 0" rpy="0 0 ${pi}" />
+      <geometry>
+        <cylinder radius="${wheel_radius}" length="${wheel_length}" />
+      </geometry>
+      <surface>
+        <friction>
+          <fdir1>1 0 0</fdir1>
+          <kp>${wheel_kp}</kp>
+          <kd>${wheel_kd}</kd>
+          <mu>${wheel_mu1}</mu>
+          <mu2>${wheel_mu2}</mu2>
+          <slip1>${wheel_slip1}</slip1>
+          <slip2>${wheel_slip2}</slip2>
+        </friction>
+      </surface>
+    </collision>
+    <inertial>
+      <mass value="${wheel_mass}" />
+      <origin xyz="0.0 0 0" rpy="0 0 ${pi}" />
       <inertia
         ixx="${wheel_inertia}" ixy="0" ixz="0"
@@ -189,5 +189,5 @@
   <link name="wheel_right_rear">
     <visual name="wheel_right_rear_visual">
-      <origin xyz="0.0 0 0" rpy="0 0 -${pi}" />
+      <origin xyz="0.0 0 0" rpy="0 0 ${pi}" />
       <geometry>
         <mesh filename="package://basketbot/meshes/wheel.dae" />
@@ -195,27 +195,87 @@
     </visual>
     <collision name="wheel_right_rear_collision">
-      <origin xyz="0.0 0 0" rpy="0 0 -${pi}" />
-      <geometry>
-        <cylinder radius="${wheel_radius}" length="${wheel_length}" />
-      </geometry>
-      <surface>
-        <friction>
-          <fdir1>1 0 0</fdir1>
-          <kp>${wheel_kp}</kp> <!-- kp and kd for rubber -->
-          <kd>${wheel_kd}</kd>
-          <mu>${wheel_mu1}</mu>
-          <mu2>${wheel_mu2}</mu2>
-          <slip1>${wheel_slip1}</slip1>
-          <slip2>${wheel_slip2}</slip2>
-        </friction>
-      </surface>
-    </collision>
-    <inertial>
-      <mass value="${wheel_mass}" />
-      <origin xyz="0.0 0 0" rpy="0 0 -${pi}" />
-      <inertia
-        ixx="${wheel_inertia}" ixy="0" ixz="0"
-        iyy="${wheel_inertia}" iyz="0"
-        izz="${wheel_inertia}"
+      <origin xyz="0.0 0 0" rpy="0 0 ${pi}" />
+      <geometry>
+        <cylinder radius="${wheel_radius}" length="${wheel_length}" />
+      </geometry>
+      <surface>
+        <friction>
+          <fdir1>1 0 0</fdir1>
+          <kp>${wheel_kp}</kp>
+          <kd>${wheel_kd}</kd>
+          <mu>${wheel_mu1}</mu>
+          <mu2>${wheel_mu2}</mu2>
+          <slip1>${wheel_slip1}</slip1>
+          <slip2>${wheel_slip2}</slip2>
+        </friction>
+      </surface>
+    </collision>
+    <inertial>
+      <mass value="${wheel_mass}" />
+      <origin xyz="0.0 0 0" rpy="0 0 ${pi}" />
+      <inertia
+        ixx="${wheel_inertia}" ixy="0" ixz="0"
+        iyy="${wheel_inertia}" iyz="0"
+        izz="${wheel_inertia}"
+      />
+    </inertial>
+  </link>
+  <!-- SENSORS  -->
+  <joint type="fixed" name="camera_joint">
+    <origin xyz=".5 0 0" rpy="0 0 0" />
+    <child link="camera" />
+    <parent link="chassis" />
+    <axis xyz="0 1 0" />
+  </joint>
+  <link name="camera">
+    <visual name="camera_visual">
+      <origin xyz="0 0 0" rpy="0 0 0"/>
+      <geometry>
+        <box size="0.05 0.05 0.05" />
+      </geometry>
+    </visual>
+    <collision name="camera_collision">
+      <origin xyz="0 0 0" rpy="0 0 0" />
+      <geometry>
+        <box size="0.05 0.05 0.05" />
+      </geometry>
+    </collision>
+    <inertial>
+      <mass value="0.1" />
+      <origin xyz="0 0 0" rpy="0 0 0" />
+      <box_inertia m="0.1" x="0.05" y="0.05" z="0.05" />
+      <inertia
+        ixx="1e-6" ixy="0" ixz="0"
+        iyy="1e-6" iyz="0"
+        izz="1e-6"
+      />
+    </inertial>
+  </link>
+  <joint type="fixed" name="hokuyo_joint">
+    <origin xyz="0.175 0 0.08" rpy="0 0 0" />
+    <child link="hokuyo" />
+    <parent link="chassis" />
+    <axis xyz="0 1 0" />
+  </joint>
+  <link name="hokuyo">
+    <visual name="hokuyo_visual">
+      <origin xyz="0 0 0" rpy="0 0 0" />
+      <geometry>
+        <mesh filename="package://basketbot/meshes/hokuyo.dae" />
+      </geometry>
+    </visual>
+    <collision name="hokuyo_collision">
+      <origin xyz="0 0 0" rpy="0 0 0" />
+      <geometry>
+        <box size="0.1 0.1 0.1" />
+      </geometry>
+    </collision>
+    <inertial>
+      <mass value="1e-5" />
+      <origin xyz="0 0 0" rpy="0 0 0" />
+      <inertia
+        ixx="1e-6" ixy="0" ixz="0"
+        iyy="1e-6" iyz="0"
+        izz="1e-6"
       />
     </inertial>

Commit message: feat: rework basketbot, ready for AMCL tweaking

File: basketbot/urdf/basketbot.xacro (robot description, xacro)
@@ -5,11 +5,11 @@
   <xacro:property name="chassis_length" value="1.1" />
   <xacro:property name="chassis_width" value="0.84" />
-  <xacro:property name="chassis_height" value="0.85" />
+  <xacro:property name="chassis_height" value="0.8" />
   <xacro:property name="wheel_length" value="0.05" />
   <xacro:property name="wheel_radius" value="0.075" />
   <xacro:property name="wheel_mass" value="0.25" />
   <xacro:property name="wheel_x_offset" value="0.35" />
-  <xacro:property name="wheel_y_offset" value="${(chassis_width/2) + (wheel_length/2)}" />
-  <xacro:property name="wheel_z_offset" value="-0.34" />
+  <xacro:property name="wheel_y_offset" value="${(chassis_width/2) + (wheel_length/2)+0.01}" />
+  <xacro:property name="wheel_z_offset" value="-${(wheel_radius)}" /> <!-- -0.355 -->
   <xacro:property name="wheel_inertia" value="0.1" />
   <xacro:property name="wheel_kp" value="1000000.0" />
@@ -27,8 +27,8 @@
   </joint>
   <link name="chassis">
-    <pose>0 0 0 0 0 0</pose>
-    <inertial>
-      <mass value="15.0" />
-      <origin xyz="0.0 0 0" rpy="0 0 0" />
+    <pose>0 0 0.1 0 0 0</pose>
+    <inertial>
+      <mass value="10.0" />
+      <origin xyz="0 0 0" rpy="0 0 0" />
       <inertia
         ixx="0.1" ixy="0" ixz="0"
@@ -38,5 +38,5 @@
     </inertial>
     <collision name="collision">
-      <origin xyz="0 0 0" rpy="0 0 0" />
+      <origin xyz="0 0 ${chassis_height/2}" rpy="0 0 0" />
       <geometry>
         <box size="${chassis_length} ${chassis_width} ${chassis_height}" />
@@ -46,5 +46,5 @@
       <origin xyz="0 0 0" rpy="0 0 0" />
       <geometry>
-      <!--<box size="${chassis_length} ${chassis_width} ${chassis_height}" />-->
+        <!--<box size="${chassis_length} ${chassis_width} ${chassis_height}" />-->
         <mesh filename="package://basketbot/meshes/BasketBotModel.dae" />
       </geometry>
@@ -53,5 +53,5 @@
   <!--  WHEELS  -->
   <joint type="continuous" name="wheel_left_front_joint">
-    <origin xyz="${wheel_x_offset} ${wheel_y_offset} ${wheel_z_offset}" rpy="0 0 0"/>
+    <origin xyz="${wheel_x_offset} ${wheel_y_offset} 0" rpy="0 0 0"/>
     <child link="wheel_left_front"/>
     <parent link="chassis"/>
@@ -61,5 +61,5 @@
   </joint>
   <joint type="continuous" name="wheel_left_rear_joint">
-    <origin xyz="-${wheel_x_offset} ${wheel_y_offset} ${wheel_z_offset}" rpy="0 0 0"/>
+    <origin xyz="-${wheel_x_offset} ${wheel_y_offset} 0" rpy="0 0 0"/>
     <child link="wheel_left_rear"/>
     <parent link="chassis"/>
@@ -69,5 +69,5 @@
   </joint>
   <joint type="continuous" name="wheel_right_front_joint">
-    <origin xyz="${wheel_x_offset} -${wheel_y_offset} ${wheel_z_offset}" rpy="0 0 0"/>
+    <origin xyz="${wheel_x_offset} -${wheel_y_offset} 0" rpy="0 0 0"/>
     <child link="wheel_right_front"/>
     <parent link="chassis"/>
@@ -77,5 +77,5 @@
   </joint>
   <joint type="continuous" name="wheel_right_rear_joint">
-    <origin xyz="-${wheel_x_offset} -${wheel_y_offset} ${wheel_z_offset}" rpy="0 0 0"/>
+    <origin xyz="-${wheel_x_offset} -${wheel_y_offset} 0" rpy="0 0 0"/>
     <child link="wheel_right_rear"/>
     <parent link="chassis"/>
@@ -86,5 +86,5 @@
   <link name="wheel_left_front">
     <visual name="wheel_left_front_visual">
-      <origin xyz="0.0 0 0" rpy="0 0 ${pi}" />
+      <origin xyz="0.0 0 -${wheel_radius}" rpy="0 0 ${pi}" />
       <geometry>
         <mesh filename="package://basketbot/meshes/wheel.dae" />
@@ -93,23 +93,23 @@
     </visual>
     <collision name="wheel_left_front_collision">
-      <origin xyz="0.0 0 0" rpy="0 0 ${pi}" />
-      <geometry>
-        <cylinder radius="${wheel_radius}" length="${wheel_length}" />
-      </geometry>
-      <surface>
-        <friction>
-          <fdir1>1 0 0</fdir1>
-          <kp>${wheel_kp}</kp>
-          <kd>${wheel_kd}</kd>
-          <mu>${wheel_mu1}</mu>
-          <mu2>${wheel_mu2}</mu2>
-          <slip1>${wheel_slip1}</slip1>
-          <slip2>${wheel_slip2}</slip2>
-        </friction>
-      </surface>
-    </collision>
-    <inertial>
-      <mass value="${wheel_mass}" />
-      <origin xyz="0.0 0 0" rpy="0 0 ${pi}" />
+      <origin xyz="0.0 0 0" rpy="0 ${pi/2} ${pi/2}" />
+      <geometry>
+        <cylinder radius="${wheel_radius}" length="${wheel_length}" />
+      </geometry>
+      <surface>
+        <friction>
+          <fdir1>1 0 0</fdir1>
+          <kp>${wheel_kp}</kp>
+          <kd>${wheel_kd}</kd>
+          <mu>${wheel_mu1}</mu>
+          <mu2>${wheel_mu2}</mu2>
+          <slip1>${wheel_slip1}</slip1>
+          <slip2>${wheel_slip2}</slip2>
+        </friction>
+      </surface>
+    </collision>
+    <inertial>
+      <mass value="${wheel_mass}" />
+      <origin xyz="0.0 0 0" rpy="0 ${pi/2} ${pi/2}" />
       <inertia
         ixx="${wheel_inertia}" ixy="0" ixz="0"
@@ -121,5 +121,5 @@
   <link name="wheel_left_rear">
     <visual name="wheel_left_rear_visual">
-      <origin xyz="0.0 0 0" rpy="0 0 ${pi}" />
+      <origin xyz="0.0 0 -${wheel_radius}" rpy="0 0 ${pi}" />
       <geometry>
         <mesh filename="package://basketbot/meshes/wheel.dae" />
@@ -127,23 +127,23 @@
     </visual>
     <collision name="wheel_left_rear_collision">
-      <origin xyz="0.0 0 0" rpy="0 0 ${pi}" />
-      <geometry>
-        <cylinder radius="${wheel_radius}" length="${wheel_length}" />
-      </geometry>
-      <surface>
-        <friction>
-          <fdir1>1 0 0</fdir1>
-          <kp>${wheel_kp}</kp>
-          <kd>${wheel_kd}</kd>
-          <mu>${wheel_mu1}</mu>
-          <mu2>${wheel_mu2}</mu2>
-          <slip1>${wheel_slip1}</slip1>
-          <slip2>${wheel_slip2}</slip2>
-        </friction>
-      </surface>
-    </collision>
-    <inertial>
-      <mass value="${wheel_mass}" />
-      <origin xyz="0.0 0 0" rpy="0 0 -${pi}" />
+      <origin xyz="0.0 0 0" rpy="0 ${pi/2} ${pi/2}" />
+      <geometry>
+        <cylinder radius="${wheel_radius}" length="${wheel_length}" />
+      </geometry>
+      <surface>
+        <friction>
+          <fdir1>1 0 0</fdir1>
+          <kp>${wheel_kp}</kp>
+          <kd>${wheel_kd}</kd>
+          <mu>${wheel_mu1}</mu>
+          <mu2>${wheel_mu2}</mu2>
+          <slip1>${wheel_slip1}</slip1>
+          <slip2>${wheel_slip2}</slip2>
+        </friction>
+      </surface>
+    </collision>
+    <inertial>
+      <mass value="${wheel_mass}" />
+      <origin xyz="0.0 0 0" rpy="0 ${pi/2} ${pi/2}" />
       <inertia
         ixx="${wheel_inertia}" ixy="0" ixz="0"
@@ -155,5 +155,5 @@
   <link name="wheel_right_front">
     <visual name="wheel_right_front_visual">
-      <origin xyz="0.0 0 0" rpy="0 0 ${pi}" />
+      <origin xyz="0.0 0 -${wheel_radius}" rpy="0 0 ${pi*2}" />
       <geometry>
       <mesh filename="package://basketbot/meshes/wheel.dae" />
@@ -161,23 +161,23 @@
     </visual>
     <collision name="wheel_right_front_collision">
-      <origin xyz="0.0 0 0" rpy="0 0 ${pi}" />
-      <geometry>
-        <cylinder radius="${wheel_radius}" length="${wheel_length}" />
-      </geometry>
-      <surface>
-        <friction>
-          <fdir1>1 0 0</fdir1>
-          <kp>${wheel_kp}</kp>
-          <kd>${wheel_kd}</kd>
-          <mu>${wheel_mu1}</mu>
-          <mu2>${wheel_mu2}</mu2>
-          <slip1>${wheel_slip1}</slip1>
-          <slip2>${wheel_slip2}</slip2>
-        </friction>
-      </surface>
-    </collision>
-    <inertial>
-      <mass value="${wheel_mass}" />
-      <origin xyz="0.0 0 0" rpy="0 0 ${pi}" />
+      <origin xyz="0.0 0 0" rpy="0 ${pi/2} ${pi/2}" />
+      <geometry>
+        <cylinder radius="${wheel_radius}" length="${wheel_length}" />
+      </geometry>
+      <surface>
+        <friction>
+          <fdir1>1 0 0</fdir1>
+          <kp>${wheel_kp}</kp>
+          <kd>${wheel_kd}</kd>
+          <mu>${wheel_mu1}</mu>
+          <mu2>${wheel_mu2}</mu2>
+          <slip1>${wheel_slip1}</slip1>
+          <slip2>${wheel_slip2}</slip2>
+        </friction>
+      </surface>
+    </collision>
+    <inertial>
+      <mass value="${wheel_mass}" />
+      <origin xyz="0.0 0 0" rpy="0 ${pi/2} ${pi/2}" />
       <inertia
         ixx="${wheel_inertia}" ixy="0" ixz="0"
@@ -189,5 +189,5 @@
   <link name="wheel_right_rear">
     <visual name="wheel_right_rear_visual">
-      <origin xyz="0.0 0 0" rpy="0 0 ${pi}" />
+      <origin xyz="0.0 0 -${wheel_radius}" rpy="0 0 ${pi*2}" />
       <geometry>
         <mesh filename="package://basketbot/meshes/wheel.dae" />
@@ -195,23 +195,23 @@
     </visual>
     <collision name="wheel_right_rear_collision">
-      <origin xyz="0.0 0 0" rpy="0 0 ${pi}" />
-      <geometry>
-        <cylinder radius="${wheel_radius}" length="${wheel_length}" />
-      </geometry>
-      <surface>
-        <friction>
-          <fdir1>1 0 0</fdir1>
-          <kp>${wheel_kp}</kp>
-          <kd>${wheel_kd}</kd>
-          <mu>${wheel_mu1}</mu>
-          <mu2>${wheel_mu2}</mu2>
-          <slip1>${wheel_slip1}</slip1>
-          <slip2>${wheel_slip2}</slip2>
-        </friction>
-      </surface>
-    </collision>
-    <inertial>
-      <mass value="${wheel_mass}" />
-      <origin xyz="0.0 0 0" rpy="0 0 ${pi}" />
+      <origin xyz="0.0 0 0" rpy="0 ${pi/2} ${pi/2}" />
+      <geometry>
+        <cylinder radius="${wheel_radius}" length="${wheel_length}" />
+      </geometry>
+      <surface>
+        <friction>
+          <fdir1>1 0 0</fdir1>
+          <kp>${wheel_kp}</kp>
+          <kd>${wheel_kd}</kd>
+          <mu>${wheel_mu1}</mu>
+          <mu2>${wheel_mu2}</mu2>
+          <slip1>${wheel_slip1}</slip1>
+          <slip2>${wheel_slip2}</slip2>
+        </friction>
+      </surface>
+    </collision>
+    <inertial>
+      <mass value="${wheel_mass}" />
+      <origin xyz="0.0 0 0" rpy="0 ${pi/2} ${pi/2}" />
       <inertia
         ixx="${wheel_inertia}" ixy="0" ixz="0"
@@ -223,5 +223,5 @@
   <!-- SENSORS  -->
   <joint type="fixed" name="camera_joint">
-    <origin xyz=".5 0 0" rpy="0 0 0" />
+    <origin xyz="0.525 0 0.2" rpy="0 0 0" />
     <child link="camera" />
     <parent link="chassis" />
@@ -253,5 +253,5 @@
   </link>
   <joint type="fixed" name="hokuyo_joint">
-    <origin xyz="0.175 0 0.08" rpy="0 0 0" />
+    <origin xyz="0.525 0 0.25" rpy="0 0 0" />
     <child link="hokuyo" />
     <parent link="chassis" />
@@ -281,3 +281,6 @@
     </inertial>
   </link>
+  <gazebo reference="camera">
+    <material>Gazebo/Red</material>
+  </gazebo>
 </robot>
